File: kicad/inzynierka/inzynierka.kicad_sch (KiCad schematic)
At the start: 17 parts

Commit message: Przypisanie footprintów
Parts:
- MICA1, MICA10, MICA11, MICA12, MICA13, MICA14, MICA15, MICA16, MICA2, MICA3, MICA4, MICA5, MICA6, MICA7, MICA8, MICA9: footprint (none) -> _moje:INMP441 breakout
- RPI-IN1: footprint (none) -> Connector_PinSocket_2.54mm:PinSocket_2x10_P2.54mm_Vertical
Changed lines of the file:
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@@
 			)
 		)
-		(property "Footprint" ""
+		(property "Footprint" "_moje:INMP441 breakout"
 			(at 139.7 38.1 0)
 			(effects
@@
 			)
 		)
-		(property "Footprint" ""
+		(property "Footprint" "_moje:INMP441 breakout"
 			(at 102.87 52.07 0)
 			(effects
@@
 			)
 		)
-		(property "Footprint" ""
+		(property "Footprint" "_moje:INMP441 breakout"
 			(at 102.87 66.04 0)
 			(effects
@@
 			)
 		)
-		(property "Footprint" ""
+		(property "Footprint" "_moje:INMP441 breakout"
 			(at 139.7 66.04 0)
 			(effects
@@
 			)
 		)
-		(property "Footprint" ""
+		(property "Footprint" "_moje:INMP441 breakout"
 			(at 102.87 24.13 0)
 			(effects
@@
 			)
 		)
-		(property "Footprint" ""
+		(property "Footprint" "_moje:INMP441 breakout"
 			(at 102.87 80.01 0)
 			(effects
@@
 			)
 		)
-		(property "Footprint" ""
+		(property "Footprint" "_moje:INMP441 breakout"
 			(at 139.7 107.95 0)
 			(effects
@@
 			)
 		)
-		(property "Footprint" ""
+		(property "Footprint" "_moje:INMP441 breakout"
 			(at 139.7 93.98 0)
 			(effects
@@
 			)
 		)
-		(property "Footprint" ""
+		(property "Footprint" "_moje:INMP441 breakout"
 			(at 139.7 80.01 0)
 			(effects
@@
 			)
 		)
-		(property "Footprint" ""
+		(property "Footprint" "Connector_PinSocket_2.54mm:PinSocket_2x10_P2.54mm_Vertical"
 			(at 250.19 127 0)
 			(effects
@@
 			)
 		)
-		(property "Footprint" ""
+		(property "Footprint" "_moje:INMP441 breakout"
 			(at 139.7 24.13 0)
 			(effects
@@
 			)
 		)
-		(property "Footprint" ""
+		(property "Footprint" "_moje:INMP441 breakout"
 			(at 139.7 52.07 0)
 			(effects
@@
 			)
 		)
-		(property "Footprint" ""
+		(property "Footprint" "_moje:INMP441 breakout"
 			(at 102.87 38.1 0)
 			(effects
@@
 			)
 		)
-		(property "Footprint" ""
+		(property "Footprint" "_moje:INMP441 breakout"
 			(at 102.87 93.98 0)
 			(effects
@@
 			)
 		)
-		(property "Footprint" ""
+		(property "Footprint" "_moje:INMP441 breakout"
 			(at 102.87 107.95 0)
 			(effects
@@
 			)
 		)
-		(property "Footprint" ""
+		(property "Footprint" "_moje:INMP441 breakout"
 			(at 102.87 121.92 0)
 			(effects
@@
 			)
 		)
-		(property "Footprint" ""
+		(property "Footprint" "_moje:INMP441 breakout"
 			(at 139.7 121.92 0)
 			(effects
